Commit message: Update lidar.xacro

File: LIDAR/lidar.xacro (robot description, xacro)
@@ -4,25 +4,70 @@
         <parent link="base_link"/>
         <child link="laser_frame"/>
-        <origin xyz="0 0 0.01" rpy="0 0 0"/>
+        <origin xyz="0.0 0 0.091" rpy="0 0 0"/>
     </joint>
     <link name="laser_frame">
-      <visual>
-        <origin xyz="0 0 0" rpy="0 0 0"/>
-        <geometry>
-          <box size="0.001 0.005 0.005"/>
-        </geometry>
-        <material name="red"/>
-      </visual>
-      <collision>
-        <origin xyz="0 0 0" rpy="0 0 0"/>
-        <geometry>
-          <box size="0.001 0.001 0.005"/>
-        </geometry>
-      </collision>
-      <inertial>
-        <mass value="0.015"/>
-        <origin xyz="0 0 0"/>
-        <inertia ixx="4.15e-6" iyy="2.407e-6" izz="2.407e-6" ixy="0" ixz="0" iyz="0"/>
-      </inertial>
+        <visual>
+            <geometry>
+                <cylinder radius="0.01" length="0.018"/>
+            </geometry>
+            <material name="red"/>
+        </visual>
+        <collision>
+            <geometry>
+                <cylinder radius="0.01" length="0.018"/>
+            </geometry>
+        </collision>
+        <xacro:inertial_cylinder mass="0.01" length="0.018" radius="0.01">
+            <origin xyz="0 0 0" rpy="0 0 0"/>
+        </xacro:inertial_cylinder>
     </link>
-</robot>
+     <gazebo reference="laser_frame">
+        <material>Gazebo/Red</material>
+        <!-- Add a ray sensor, and give it a name -->
+        <sensor name="laser" type="ray">
+            <pose> 0 0 0 0 0 0 </pose>
+             <!-- Enable visualization to see the rays in the GUI -->
+            <visualize>true</visualize>
+            <!-- Set the update rate of the sensor -->
+            <update_rate>30</update_rate>
+            <ray>
+             <!-- The scan element contains the horizontal and vertical beams.
+       We are leaving out the vertical beams for this tutorial. -->
+                <scan>
+                <!-- The horizontal beams -->
+                    <horizontal>
+                     <!-- The velodyne has 32 beams(samples) -->
+                        <samples>32</samples>
+                      <!-- Resolution is multiplied by samples to determine number of
+           simulated beams vs interpolated beams. See:
+           http://sdformat.org/spec?ver=1.6&elem=sensor#horizontal_resolution
+           -->
+                        <resolution>1</resolution>
+                        <!-- Minimum angle in radians -->
+                        <min_angle>-0.53529248</min_angle>
+                        <!-- Maximum angle in radians -->
+                        <max_angle>0.18622663</max_angle>
+                    </horizontal>
+                </scan>
+                <range>
+                 <!-- Minimum distance of the beam -->
+                    <min>0.1</min>
+                    <!-- Maximum distance of the beam -->
+                    <max>3</max>
+                </range>
+                <!-- Use gaussian noise
+                <noise>
+                <type>gaussian</type>
+                  <mean>0.0</mean>
+                  <stddev>0.02</stddev>
+                </noise>-->
+            </ray>
+            <plugin name="laser_controller" filename="libgazebo_ros_laser.so">
+            <gaussianNoise>0.005</gaussianNoise>
+            <alwaysOn>true</alwaysOn>
+            <updateRate>30.0</updateRate>
+            <topicName>ray_scan</topicName>
+            <frameName>laser_frame</frameName>
+        </plugin>
+        </sensor>
+    </gazebo>
