Commit message: Add files via upload

File: LIDAR/clover4.xacro (robot description, xacro)
@@ -7,5 +7,4 @@
   <xacro:arg name="maintain_camera_rate" default="false"/>
   <xacro:arg name="use_clover_physics" default="false"/>
-  <xacro:arg name="mavlink_tcp_port" default="4560"/>
   <xacro:include filename="clover4_base.xacro" />
   <xacro:include filename="../sensors/rpi_cam.urdf.xacro"/>
@@ -14,5 +13,9 @@
   <!-- Create camera plugin -->
   <xacro:if value="$(arg main_camera)">
-    <xacro:rpi_cam name="main_camera" parent="base_link" x="0.055" y="0.0" z="-0.03" roll="0" pitch="${pi/2}" yaw="0" width="320" height="240" rate="40" do_throttling="$(arg maintain_camera_rate)"/>
+    <xacro:rpi_cam name="main_camera" parent="base_link" x="0.055" y="0.0" z="-0.03" roll="0" pitch="${pi / 2}" yaw="0" width="320" height="240" rate="40" do_throttling="$(arg maintain_camera_rate)"/>
+  </xacro:if>
+  <!-- Create rangefinder plugin -->
+  <xacro:if value="$(arg rangefinder)">
+    <xacro:distance_sensor parent="base_link" x="0.0" y="0.0" z="-0.04" roll="0" pitch="${pi / 2}" yaw="0"/>
   </xacro:if>
   <!-- Instantiate LED strip -->
@@ -21,13 +24,9 @@
       name="led"
       parent="base_link"
-      radius="0.1"
-      bulb_radius="0.01"
-      led_count="72"
+      radius="0.08"
+      bulb_radius="0.006"
+      led_count="58"
       use_plugin="true"
       z="-0.002"/>
-  </xacro:if>
-  <!-- Create rangefinder plugin -->
-  <xacro:if value="$(arg rangefinder)">
-    <xacro:distance_sensor parent="base_link" x="0.0" y="0.0" z="-0.04" roll="0" pitch="${pi / 2}" yaw="0"/>
   </xacro:if>
   <xacro:if value="$(arg gps)">
@@ -44,4 +43,4 @@
     </gazebo>
   </xacro:if>
-   <xacro:include filename="lidar.xacro" />
+  <xacro:include filename="lidar.xacro" />
 </robot>

File: LIDAR/lidar.xacro (robot description, xacro)
@@ -1,4 +1,5 @@
 <?xml version="1.0"?>
 <robot xmlns:xacro="http://www.ros.org/wiki/xacro" >
+<!-- per oleg, just attached directly to base_link
     <joint name="laser_joint" type="fixed">
         <parent link="base_link"/>
@@ -18,9 +19,10 @@
             </geometry>
         </collision>
-        <xacro:inertial_cylinder mass="0.01" length="0.018" radius="0.01">
+        <xacro:inertial_cylinder mass="0.0001" length="0.018" radius="0.01">
             <origin xyz="0 0 0" rpy="0 0 0"/>
         </xacro:inertial_cylinder>
-    </link>
-     <gazebo reference="laser_frame">
+    </link>-->
+     <!--<gazebo reference="laser_frame">-->
+     <gazebo reference="base_link">
         <material>Gazebo/Red</material>
         <!-- Add a ray sensor, and give it a name -->
@@ -45,14 +47,14 @@
                         <resolution>1</resolution>
                         <!-- Minimum angle in radians -->
-                        <min_angle>-0.53529248</min_angle>
+                        <min_angle>-0.785398</min_angle>
                         <!-- Maximum angle in radians -->
-                        <max_angle>0.18622663</max_angle>
+                        <max_angle>0.785398</max_angle>
                     </horizontal>
                 </scan>
                 <range>
                  <!-- Minimum distance of the beam -->
-                    <min>0.1</min>
+                    <min>0.3</min>
                     <!-- Maximum distance of the beam -->
-                    <max>3</max>
+                    <max>4</max>
                 </range>
                 <!-- Use gaussian noise
@@ -72,2 +74,3 @@
         </sensor>
     </gazebo>
+</robot>
